Commit message: fix controllers

File: description/camera.xacro (robot description, xacro)
@@ -34,7 +34,9 @@
         <material>Gazebo/Black</material>
         <sensor name="camera" type="camera">
-            <pose> 0 0 0 0 0 0 </pose>
+            <pose>0 0 0 0 0 0</pose>
             <visualize>true</visualize>
             <update_rate>10</update_rate>
+            <!-- gz topic name — must match the bridge arg in launch_sim.launch.py -->
+            <topic>/camera/image_raw</topic>
             <camera>
                 <!-- {to change} -->
@@ -51,9 +53,4 @@
                 </clip>
             </camera>
-            <plugin filename="gz_ros2_camera-system" name="camera_plugin">
-                <frame_name>camera_link_optical</frame_name>
-                <topic>/camera/image_raw</topic>
-                <camera_name>camera1</camera_name>
-            </plugin>
         </sensor>
     </gazebo>

File: description/robot_core.xacro (robot description, xacro)
@@ -33,15 +33,12 @@
         <color rgba="1 0 0 1"/>
     </material>
+  <!-- ===== ROOT LINK ===== -->
+  <link name="base_link"/>
+  <joint name="base_link_chassis_joint" type="fixed">
+    <parent link="base_link"/>
+    <child link="chassis"/>
+    <origin xyz="0 0 0.115" rpy="0 0 0"/>
+  </joint>
   <!-- ===== BASE LINK: CHASSIS ===== -->
-    <!--
-        BASE_FOOTPRINT LINK
-      <joint name="base_footprint_joint" type="fixed">
-          <parent link="base_link"/>
-          <child link="base_footprint"/>
-          <origin xyz="0 0 0" rpy="0 0 0"/>
-      </joint>
-      <link name="base_footprint">
-      </link>
-    -->
   <link name="chassis">
     <visual>

File: description/ros2_control.xacro (robot description, xacro)
@@ -61,7 +61,11 @@
     </xacro:if>
     <gazebo>
-        <plugin filename="gz_ros2_control-system" name="gz_ros2_control::GazeboSimROS2ControlPlugin">
+        <plugin filename="gz_ros2_control-system"
+                name="gz_ros2_control::GazeboSimROS2ControlPlugin">
             <parameters>$(find grad-project)/config/my_controllers.yaml</parameters>
             <parameters>$(find grad-project)/config/gaz_ros2_ctl_use_sim.yaml</parameters>
+            <!-- FIX: auto-activate controllers on robot spawn -->
+            <controller_manager_prefix_node_name>controller_manager</controller_manager_prefix_node_name>
+            <activate_controllers_on_start>diff_cont joint_broad</activate_controllers_on_start>
         </plugin>
     </gazebo>

Commit message: ros2_control, Gazebo, Keyboard control, works as expected

File: description/camera.xacro (robot description, xacro)
@@ -37,5 +37,4 @@
             <visualize>true</visualize>
             <update_rate>10</update_rate>
-            <!-- gz topic name — must match the bridge arg in launch_sim.launch.py -->
             <topic>/camera/image_raw</topic>
             <camera>

File: description/robot.urdf.xacro (robot description, xacro)
@@ -1,5 +1,5 @@
 <?xml version="1.0" encoding="utf-8"?>
 <robot xmlns:xacro="http://www.ros.org/wiki/xacro"  name="amr">
-    <xacro:arg name="sim_mode" default="True"/>
+    <xacro:arg name="sim_mode" default="False"/>
     <xacro:include filename="robot_core.xacro" />
     <xacro:include filename="camera.xacro" />

File: description/robot_core.xacro (robot description, xacro)
@@ -1,5 +1,4 @@
 <?xml version="1.0" encoding="utf-8"?>
 <robot xmlns:xacro="http://www.ros.org/wiki/xacro">
-    <!-- <xacro:include filename="inertial_macros.xacro"/> -->
     <xacro:property name="chassis_length" value="0.4"/>
     <xacro:property name="chassis_width" value="0.3"/>
@@ -10,7 +9,7 @@
     <xacro:property name="wheel_mass" value="0.5"/>
     <!--
-    <xacro:property name="wheel_offset_x" value="0.226"/>
-    <xacro:property name="wheel_offset_y" value="0.1485"/>
-    <xacro:property name="wheel_offset_z" value="0.01"/>
+    <xacro:property name="wheel_offset_x" value=""/>
+    <xacro:property name="wheel_offset_y" value=""/>
+    <xacro:property name="wheel_offset_z" value=""/>
     -->
   <!-- ===== MATERIALS ===== -->
@@ -56,12 +55,8 @@
       <origin xyz="0 0 0" rpy="0 0 0"/>
       <mass value="${chassis_mass}"/>
-      <!-- Inertia for a uniform box: Ixx = (m/12)*(y^2+z^2), etc. -->
       <inertia ixx="0.09375" ixy="0.0" ixz="0.0"
                iyy="0.15208" iyz="0.0"
                izz="0.20833"/>
     </inertial>
-    <!-- <xacro:inertial_box mass="0.5" x="${chassis_length}" y="${chassis_width}" z="${chassis_height}">
-            <origin xyz="${chassis_length/2} 0 ${chassis_height/2}" rpy="0 0 0"/>
-         </xacro:inertial_box> -->
   </link>
     <gazebo reference="chassis">
@@ -85,18 +80,14 @@
       <origin xyz="0 0 0" rpy="0 0 0"/>
       <mass value="${wheel_mass}"/>
-      <!-- Cylinder axis along y: Iyy = 0.5*m*r^2, Ixx = Izz = (m/12)*(3r^2 + L^2) -->
       <inertia ixx="0.0004875" ixy="0.0" ixz="0.0"
                iyy="0.0009"    iyz="0.0"
                izz="0.0004875"/>
     </inertial>
-    <!-- <xacro:inertial_cylinder mass="${wheel_mass}" length="${wheel_thickness}" radius="${wheel_radius}">
-            <origin xyz="0 0 0" rpy="0 0 0"/>
-         </xacro:inertial_cylinder> -->
   </link>
   <joint name="left_wheel_joint" type="continuous">
     <parent link="chassis"/>
     <child link="left_wheel"/>
-    <origin xyz="0 -0.165 -0.055" rpy="-${pi/2} 0 0"/>
-    <axis xyz="0 0 -1"/>
+    <origin xyz="0 -0.165 -0.055" rpy="${pi/2} 0 0"/>
+    <axis xyz="0 0 1"/>
   </joint>
   <gazebo reference="left_wheel">
@@ -123,7 +114,4 @@
                izz="0.0004875"/>
     </inertial>
-    <!-- <xacro:inertial_cylinder mass="${wheel_mass}" length="${wheel_thickness}" radius="${wheel_radius}">
-            <origin xyz="0 0 0" rpy="0 0 0"/>
-         </xacro:inertial_cylinder> -->
   </link>
   <joint name="right_wheel_joint" type="continuous">
@@ -131,9 +119,8 @@
     <child link="right_wheel"/>
     <origin xyz="0 0.165 -0.055" rpy="${pi/2} 0 0"/>
-    <!-- <origin xyz="0 ${wheel_offset_y} 0" rpy="${pi/2} 0 0" /> -->
-    <axis xyz="0 0 -1"/>
+    <axis xyz="0 0 1"/>
   </joint>
   <gazebo reference="right_wheel">
-      <material>Ignition/Blue</material>
+      <material>Gazebo/Blue</material>
   </gazebo>
   <!-- ===== SUPPORT WHEELS (casters, modeled as spheres) ===== -->
@@ -154,5 +141,4 @@
       <origin xyz="0 0 0" rpy="0 0 0"/>
       <mass value="0.1"/>
-      <!-- Solid sphere inertia: (2/5)*m*r^2 -->
       <inertia ixx="0.000016" ixy="0.0" ixz="0.0"
                iyy="0.000016" iyz="0.0"
@@ -165,4 +151,8 @@
     <origin xyz="0.2 0.15 -0.095" rpy="0 0 0"/>
   </joint>
+  <gazebo reference="support_front_left">
+    <mu1>0.01</mu1>
+    <mu2>0.01</mu2>
+  </gazebo>
   <!-- Front right corner (x = +0.2, y = -0.15) -->
   <link name="support_front_right">
@@ -191,4 +181,8 @@
     <origin xyz="0.2 -0.15 -0.095" rpy="0 0 0"/>
   </joint>
+  <gazebo reference="support_front_right">
+    <mu1>0.01</mu1>
+    <mu2>0.01</mu2>
+  </gazebo>
   <!-- Back left corner (x = -0.2, y = +0.15) -->
   <link name="support_back_left">
@@ -217,4 +211,8 @@
     <origin xyz="-0.2 0.15 -0.095" rpy="0 0 0"/>
   </joint>
+  <gazebo reference="support_back_left">
+    <mu1>0.01</mu1>
+    <mu2>0.01</mu2>
+  </gazebo>
   <!-- Back right corner (x = -0.2, y = -0.15) -->
   <link name="support_back_right">
@@ -243,3 +241,7 @@
     <origin xyz="-0.2 -0.15 -0.095" rpy="0 0 0"/>
   </joint>
+  <gazebo reference="support_back_right">
+    <mu1>0.01</mu1>
+    <mu2>0.01</mu2>
+  </gazebo>
 </robot>
