Commit message: =

File: description/camera.xacro (robot description, xacro)
@@ -4,23 +4,19 @@
         <parent link="chassis"/>
         <child link="camera_link"/>
-        <!-- {to change} -->
-        <origin xyz="0.276 0 0.181" rpy="0 0.18 0"/>
-        <!-- {end changes} -->
+        <origin xyz="0.126 -0.066 0.0435" rpy="0 0 0"/>
     </joint>
     <link name="camera_link">
         <visual>
             <geometry>
-                <!-- {to change} -->
-                <box size="0.010 0.03 0.03"/>
-                <!-- {end changes} -->
+                <box size="0.01 0.04 0.025"/>
             </geometry>
-            <material name="black"/>
+            <material name="blue"/>
         </visual>
         <visual>
-            <origin xyz="0 0 -0.05"/>
+            <origin xyz="0.005 -0.011 0" rpy="0 ${-pi/2} 0"/>
             <geometry>
-                <cylinder radius="0.002" length="0.1"/>
+                <cylinder radius="0.004" length="0.01"/>
             </geometry>
-            <material name="black"/>
+            <material name="blue"/>
         </visual>
     </link>
@@ -28,5 +24,5 @@
         <parent link="camera_link"/>
         <child link="camera_link_optical"/>
-        <origin xyz="0 0 0" rpy="${-pi/2} 0 ${-pi/2}"/>
+        <origin xyz="0.005 -0.011 0" rpy="${-pi/2}  0 ${-pi/2}"/>
     </joint>
     <link name="camera_link_optical"></link>

File: description/robot.urdf.xacro (robot description, xacro)
@@ -2,4 +2,5 @@
 <robot xmlns:xacro="http://www.ros.org/wiki/xacro"  name="amr">
     <xacro:arg name="sim_mode" default="False"/>
+    <xacro:include filename="inertial_macros.xacro" />
     <xacro:include filename="robot_core.xacro" />
     <xacro:include filename="camera.xacro" />

File: description/robot_core.xacro (robot description, xacro)
@@ -1,17 +1,30 @@
 <?xml version="1.0" encoding="utf-8"?>
 <robot xmlns:xacro="http://www.ros.org/wiki/xacro">
-    <xacro:property name="chassis_length" value="0.4"/>
-    <xacro:property name="chassis_width" value="0.3"/>
-    <xacro:property name="chassis_height" value="0.15"/>
-    <xacro:property name="chassis_mass" value="10.0"/>
-    <xacro:property name="wheel_radius" value="0.06"/>
-    <xacro:property name="wheel_thickness" value="0.03"/>
-    <xacro:property name="wheel_mass" value="0.5"/>
-    <!--
-    <xacro:property name="wheel_offset_x" value=""/>
-    <xacro:property name="wheel_offset_y" value=""/>
-    <xacro:property name="wheel_offset_z" value=""/>
-    -->
-  <!-- ===== MATERIALS ===== -->
+  <!-- ============================================================ -->
+  <!--  ROBOT PROPERTIES                                            -->
+  <!-- ============================================================ -->
+  <xacro:property name="chassis_length"  value="0.27" />
+  <xacro:property name="chassis_width"   value="0.18" />
+  <xacro:property name="chassis_height"  value="0.127" />
+  <xacro:property name="chassis_mass"    value="1.5" />
+  <xacro:property name="wheel_radius"    value="0.033" />
+  <xacro:property name="wheel_thickness" value="0.03" />
+  <xacro:property name="wheel_mass"      value="0.05" />
+  <!-- Wheel positions relative to chassis frame (at chassis centre) -->
+  <xacro:property name="wheel_x" value="0.0" />
+  <xacro:property name="wheel_y" value="0.09" />
+  <xacro:property name="wheel_z" value="-0.0705" />
+  <xacro:property name="support_radius"  value="0.014" />
+  <xacro:property name="support_mass"    value="0.05" />
+  <xacro:property name="support_x"       value="0.121" />
+  <xacro:property name="support_y"       value="0.076" />
+  <xacro:property name="support_z"       value="-0.0895" />
+  <xacro:property name="imu_mass"  value="0.01" />
+  <xacro:property name="imu_size"  value="0.02" />
+  <!-- The robot's base link is placed at the ground contact point -->
+  <xacro:property name="base_z_offset" value="0.0" />
+  <!-- ============================================================ -->
+  <!--  MATERIALS                                                   -->
+  <!-- ============================================================ -->
   <material name="grey">
     <color rgba="0.5 0.5 0.5 1.0"/>
@@ -20,248 +33,177 @@
     <color rgba="0.1 0.1 0.1 1.0"/>
   </material>
-    <material name="white">
-        <color rgba="1 1 1 1" />
-    </material>
-    <material name="orange">
-        <color rgba="1 0.3 0.1 1"/>
-    </material>
-    <material name="blue">
-        <color rgba="0.2 0.2 1 1"/>
-    </material>
-    <material name="red">
-        <color rgba="1 0 0 1"/>
-    </material>
-  <!-- ===== ROOT LINK ===== -->
-  <link name="base_link"></link>
+  <material name="white">
+    <color rgba="1 1 1 1" />
+  </material>
+  <material name="orange">
+    <color rgba="1 0.3 0.1 1"/>
+  </material>
+  <material name="blue">
+    <color rgba="0.2 0.2 1 1"/>
+  </material>
+  <material name="red">
+    <color rgba="1 0 0 1"/>
+  </material>
+  <!-- ============================================================ -->
+  <!--  BASE LINKS AND ROOT                                         -->
+  <!-- ============================================================ -->
+  <!-- The base_footprint is the virtual ground contact point -->
+  <link name="base_footprint" />
+  <joint name="base_footprint_joint" type="fixed">
+    <parent link="base_footprint" />
+    <child link="base_link" />
+    <origin xyz="0 0 ${base_z_offset}" rpy="0 0 0" />
+  </joint>
+  <!-- The base_link is the main frame, located at the chassis centre height? -->
+  <!-- We'll place base_link at the chassis centre to simplify transforms. -->
+  <!-- But original had base_link at (0,0,0) and chassis joint offset. We'll keep that -->
+  <!-- for compatibility: base_link is at (0,0,0) and chassis is offset. -->
+  <!-- However, we now have base_footprint at ground, and base_link at z=0. So chassis -->
+  <!-- centre is at z=0.115, as before. -->
+  <link name="base_link" />
+  <!-- ============================================================ -->
+  <!--  CHASSIS                                                     -->
+  <!-- ============================================================ -->
   <joint name="base_link_chassis_joint" type="fixed">
-    <parent link="base_link"/>
-    <child link="chassis"/>
-    <origin xyz="0 0 0.115" rpy="0 0 0"/>
+    <parent link="base_link" />
+    <child link="chassis" />
+    <origin xyz="0 0 ${chassis_height/2 + 0.04}" rpy="0 0 0" />
   </joint>
-  <!-- ===== BASE LINK: CHASSIS ===== -->
   <link name="chassis">
     <visual>
       <geometry>
-        <box size="${chassis_length} ${chassis_width} ${chassis_height}"/>
-      </geometry>
-      <material name="grey"/>
+        <box size="${chassis_length} ${chassis_width} ${chassis_height}" />
+      </geometry>
+      <material name="grey" />
     </visual>
     <collision>
       <geometry>
-        <box size="0.4 0.3 0.15"/>
+        <box size="${chassis_length} ${chassis_width} ${chassis_height}" />
       </geometry>
     </collision>
-    <inertial>
+    <xacro:inertial_box mass="${chassis_mass}"
+                        x="${chassis_length}"
+                        y="${chassis_width}"
+                        z="${chassis_height}">
       <origin xyz="0 0 0" rpy="0 0 0"/>
-      <mass value="${chassis_mass}"/>
-      <inertia ixx="0.09375" ixy="0.0" ixz="0.0"
-               iyy="0.15208" iyz="0.0"
-               izz="0.20833"/>
-    </inertial>
+    </xacro:inertial_box>
   </link>
-    <gazebo reference="chassis">
-        <material>Gazebo/Orange</material>
+  <gazebo reference="chassis">
+    <material>Gazebo/Orange</material>
+  </gazebo>
+  <!-- ============================================================ -->
+  <!--  MACRO: CREATE A DRIVE WHEEL                                 -->
+  <!-- ============================================================ -->
+  <xacro:macro name="drive_wheel" params="name side x y z">
+    <!-- side: 'left' or 'right' to set joint axis sign? Actually we use same axis, -->
+    <!-- but we can set different orientation? No, we keep same. -->
+    <link name="${name}_wheel">
+      <visual>
+        <geometry>
+          <cylinder radius="${wheel_radius}" length="${wheel_thickness}" />
+        </geometry>
+        <material name="black" />
+      </visual>
+      <collision>
+        <geometry>
+          <cylinder radius="${wheel_radius}" length="${wheel_thickness}" />
+        </geometry>
+      </collision>
+      <xacro:inertial_cylinder mass="${wheel_mass}"
+                               length="${wheel_thickness}"
+                               radius="${wheel_radius}" >
+        <origin xyz="0 0 0" rpy="0 0 0"/>
+      </xacro:inertial_cylinder>
+    </link>
+    <joint name="${name}_wheel_joint" type="fixed">
+      <parent link="chassis" />
+      <child link="${name}_wheel" />
+      <!-- The wheel is rotated so its axis aligns with Y (roll direction) -->
+      <origin xyz="${x} ${y} ${z}" rpy="${pi/2} 0 0" />
+      <axis xyz="0 0 1" />
+      <dynamics damping="0.0" friction="0.0" />
+    </joint>
+    <gazebo reference="${name}_wheel">
+      <material>Gazebo/Blue</material>
+      <mu1>0.8</mu1>
+      <mu2>0.8</mu2>
+      <friction>1.0</friction>
     </gazebo>
- <!-- ===== DRIVE WHEELS ===== -->
-  <!-- Left drive wheel -->
-  <link name="left_wheel">
+  </xacro:macro>
+  <!-- Instantiate the two drive wheels -->
+  <xacro:drive_wheel name="left"  side="left"  x="${wheel_x}" y="-${wheel_y}" z="${wheel_z}" />
+  <xacro:drive_wheel name="right" side="right" x="${wheel_x}" y="${wheel_y}"  z="${wheel_z}" />
+  <!-- ============================================================ -->
+  <!--  MACRO: CREATE A SUPPORT CASTER (sphere)                     -->
+  <!-- ============================================================ -->
+  <xacro:macro name="support_caster" params="name x y z">
+    <link name="support_${name}">
+      <visual name="support_caster">
+        <origin xyz="0 0 0" rpy="0 0 0"/>
+        <geometry>
+          <sphere radius="${support_radius}" />
+        </geometry>
+        <material name="black" />
+      </visual>
+      <visual name="support_caster_stand">
+        <origin xyz="0 0 0.02" rpy="0 0 ${-pi/2}"/>
+        <geometry>
+          <cylinder radius="0.01" length="0.014"/>
+        </geometry>
+        <material name="black"/>
+      </visual>
+      <collision>
+        <geometry>
+          <sphere radius="${support_radius}" />
+        </geometry>
+      </collision>
+      <xacro:inertial_sphere mass="${support_mass}"
+                             radius="${support_radius}" >
+        <origin xyz="0 0 0" rpy="0 0 0"/>
+      </xacro:inertial_sphere>
+    </link>
+    <joint name="support_${name}_joint" type="fixed">
+      <parent link="chassis" />
+      <child link="support_${name}" />
+      <origin xyz="${x} ${y} ${z}" rpy="0 0 0" />
+    </joint>
+    <gazebo reference="support_${name}">
+      <mu1>0.01</mu1>
+      <mu2>0.01</mu2>
+      <friction>0.01</friction>
+    </gazebo>
+  </xacro:macro>
+  <!-- Four corners -->
+  <xacro:support_caster name="front_left"  x="${support_x}"  y="${support_y}"  z="${support_z}" />
+  <xacro:support_caster name="front_right" x="${support_x}"  y="-${support_y}" z="${support_z}" />
+  <xacro:support_caster name="back_left"   x="-${support_x}" y="${support_y}"  z="${support_z}" />
+  <xacro:support_caster name="back_right"  x="-${support_x}" y="-${support_y}" z="${support_z}" />
+  <!-- ============================================================ -->
+  <!--  IMU SENSOR                                                  -->
+  <!-- ============================================================ -->
+  <link name="imu_link">
     <visual>
       <geometry>
-        <cylinder radius="${wheel_radius}" length="${wheel_thickness}"/>
-      </geometry>
-      <material name="black"/>
+        <box size="${imu_size} ${imu_size} ${imu_size/4}" />
+      </geometry>
+      <material name="white" />
     </visual>
     <collision>
       <geometry>
-        <cylinder radius="${wheel_radius}" length="${wheel_thickness}"/>
+        <box size="${imu_size} ${imu_size} ${imu_size/4}" />
       </geometry>
     </collision>
-    <inertial>
+    <xacro:inertial_box mass="${imu_mass}"
+                        x="${imu_size}"
+                        y="${imu_size}"
+                        z="${imu_size/2.5}" >
       <origin xyz="0 0 0" rpy="0 0 0"/>
-      <mass value="${wheel_mass}"/>
-      <inertia ixx="0.0004875" ixy="0.0" ixz="0.0"
-               iyy="0.0009"    iyz="0.0"
-               izz="0.0004875"/>
-    </inertial>
+    </xacro:inertial_box>
   </link>
-  <joint name="left_wheel_joint" type="continuous">
-    <parent link="chassis"/>
-    <child link="left_wheel"/>
-    <origin xyz="0 -0.165 -0.055" rpy="${pi/2} 0 0"/>
-    <axis xyz="0 0 1"/>
+  <joint name="imu_joint" type="fixed">
+    <parent link="base_link" />
+    <child link="imu_link" />
+    <origin xyz="0 0 ${chassis_height + 0.034}" rpy="0 0 0" />
   </joint>
-  <gazebo reference="left_wheel">
-      <material>Gazebo/Blue</material>
-  </gazebo>
- <!-- Right drive wheel -->
-  <link name="right_wheel">
-    <visual>
-      <geometry>
-        <cylinder radius="${wheel_radius}" length="${wheel_thickness}"/>
-      </geometry>
-      <material name="black"/>
-    </visual>
-    <collision>
-      <geometry>
-        <cylinder radius="${wheel_radius}" length="${wheel_thickness}"/>
-      </geometry>
-    </collision>
-    <inertial>
-      <origin xyz="0 0 0" rpy="0 0 0"/>
-      <mass value="${wheel_mass}"/>
-      <inertia ixx="0.0004875" ixy="0.0" ixz="0.0"
-               iyy="0.0009"    iyz="0.0"
-               izz="0.0004875"/>
-    </inertial>
-  </link>
-  <joint name="right_wheel_joint" type="continuous">
-    <parent link="chassis"/>
-    <child link="right_wheel"/>
-    <origin xyz="0 0.165 -0.055" rpy="${pi/2} 0 0"/>
-    <axis xyz="0 0 1"/>
-  </joint>
-  <gazebo reference="right_wheel">
-      <material>Gazebo/Blue</material>
-  </gazebo>
-  <!-- ===== SUPPORT WHEELS (casters, modeled as spheres) ===== -->
-  <!-- Front left corner (x = +0.2, y = +0.15) -->
-  <link name="support_front_left">
-    <visual>
-      <geometry>
-        <sphere radius="0.02"/>
-      </geometry>
-      <material name="black"/>
-    </visual>
-    <collision>
-      <geometry>
-        <sphere radius="0.02"/>
-      </geometry>
-    </collision>
-    <inertial>
-      <origin xyz="0 0 0" rpy="0 0 0"/>
-      <mass value="0.1"/>
-      <inertia ixx="0.000016" ixy="0.0" ixz="0.0"
-               iyy="0.000016" iyz="0.0"
-               izz="0.000016"/>
-    </inertial>
-  </link>
-  <joint name="support_front_left_joint" type="fixed">
-    <parent link="chassis"/>
-    <child link="support_front_left"/>
-    <origin xyz="0.2 0.15 -0.095" rpy="0 0 0"/>
-  </joint>
-  <gazebo reference="support_front_left">
-    <mu1>0.01</mu1>
-    <mu2>0.01</mu2>
-  </gazebo>
-  <!-- Front right corner (x = +0.2, y = -0.15) -->
-  <link name="support_front_right">
-    <visual>
-      <geometry>
-        <sphere radius="0.02"/>
-      </geometry>
-      <material name="black"/>
-    </visual>
-    <collision>
-      <geometry>
-        <sphere radius="0.02"/>
-      </geometry>
-    </collision>
-    <inertial>
-      <origin xyz="0 0 0" rpy="0 0 0"/>
-      <mass value="0.1"/>
-      <inertia ixx="0.000016" ixy="0.0" ixz="0.0"
-               iyy="0.000016" iyz="0.0"
-               izz="0.000016"/>
-    </inertial>
-  </link>
-  <joint name="support_front_right_joint" type="fixed">
-    <parent link="chassis"/>
-    <child link="support_front_right"/>
-    <origin xyz="0.2 -0.15 -0.095" rpy="0 0 0"/>
-  </joint>
-  <gazebo reference="support_front_right">
-    <mu1>0.01</mu1>
-    <mu2>0.01</mu2>
-  </gazebo>
-  <!-- Back left corner (x = -0.2, y = +0.15) -->
-  <link name="support_back_left">
-    <visual>
-      <geometry>
-        <sphere radius="0.02"/>
-      </geometry>
-      <material name="black"/>
-    </visual>
-    <collision>
-      <geometry>
-        <sphere radius="0.02"/>
-      </geometry>
-    </collision>
-    <inertial>
-      <origin xyz="0 0 0" rpy="0 0 0"/>
-      <mass value="0.1"/>
-      <inertia ixx="0.000016" ixy="0.0" ixz="0.0"
-               iyy="0.000016" iyz="0.0"
-               izz="0.000016"/>
-    </inertial>
-  </link>
-  <joint name="support_back_left_joint" type="fixed">
-    <parent link="chassis"/>
-    <child link="support_back_left"/>
-    <origin xyz="-0.2 0.15 -0.095" rpy="0 0 0"/>
-  </joint>
-  <gazebo reference="support_back_left">
-    <mu1>0.01</mu1>
-    <mu2>0.01</mu2>
-  </gazebo>
-  <!-- Back right corner (x = -0.2, y = -0.15) -->
-  <link name="support_back_right">
-    <visual>
-      <geometry>
-        <sphere radius="0.02"/>
-      </geometry>
-      <material name="black"/>
-    </visual>
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
File: description/ros2_control.xacro (robot description, xacro)
@@ -2,29 +2,27 @@
 <robot xmlns:xacro="http://www.ros.org/wiki/xacro">
   <xacro:unless value="$(arg sim_mode)">
-    <ros2_control name="Esp32DiffDrive" type="system">
-      <hardware>
-        <plugin>esp32_diff_hw_interface/Esp32DiffHwInterface</plugin>
-        <!--
-        <param name="left_wheel_name">left_wheel_joint</param>
-        <param name="right_wheel_name">right_wheel_joint</param>
-        -->
-      </hardware>
-      <joint name="left_wheel_joint">
-        <command_interface name="velocity">
-          <param name="min">-10.0</param>
-          <param name="max"> 10.0</param>
-        </command_interface>
-        <state_interface name="position"/>
-        <state_interface name="velocity"/>
-      </joint>
-      <joint name="right_wheel_joint">
-        <command_interface name="velocity">
-          <param name="min">-10.0</param>
-          <param name="max"> 10.0</param>
-        </command_interface>
-        <state_interface name="position"/>
-        <state_interface name="velocity"/>
-      </joint>
-    </ros2_control>
+<ros2_control name="EspDiffDrive" type="system">
+  <hardware>
+    <plugin>esp_diff_interface/esp_diff</plugin>
+    <param name="left_wheel_name">left_wheel_joint</param>
+    <param name="right_wheel_name">right_wheel_joint</param>
+  </hardware>
+  <joint name="left_wheel_joint">
+    <command_interface name="velocity">
+      <param name="min">-0.7</param>
+      <param name="max">0.7</param>
+    </command_interface>
+    <state_interface name="position"/>
+    <state_interface name="velocity"/>
+  </joint>
+  <joint name="right_wheel_joint">
+    <command_interface name="velocity">
+      <param name="min">-0.7</param>
+      <param name="max">0.7</param>
+    </command_interface>
+    <state_interface name="position"/>
+    <state_interface name="velocity"/>
+  </joint>
+</ros2_control>
   </xacro:unless>
   <xacro:if value="$(arg sim_mode)">
