Commit message: fix the diff drive manager

File: description/robot_core.xacro (robot description, xacro)
@@ -34,5 +34,5 @@
     </material>
   <!-- ===== ROOT LINK ===== -->
-  <link name="base_link"/>
+  <link name="base_link"></link>
   <joint name="base_link_chassis_joint" type="fixed">
     <parent link="base_link"/>
@@ -66,5 +66,5 @@
   </link>
     <gazebo reference="chassis">
-        <material>Ignition/Orange</material>
+        <material>Gazebo/Orange</material>
     </gazebo>
  <!-- ===== DRIVE WHEELS ===== -->
@@ -98,8 +98,8 @@
     <child link="left_wheel"/>
     <origin xyz="0 -0.165 -0.055" rpy="-${pi/2} 0 0"/>
-    <axis xyz="0 1 0"/>
+    <axis xyz="0 0 -1"/>
   </joint>
   <gazebo reference="left_wheel">
-      <material>Ignition/Blue</material>
+      <material>Gazebo/Blue</material>
   </gazebo>
  <!-- Right drive wheel -->
@@ -132,5 +132,5 @@
     <origin xyz="0 0.165 -0.055" rpy="${pi/2} 0 0"/>
     <!-- <origin xyz="0 ${wheel_offset_y} 0" rpy="${pi/2} 0 0" /> -->
-    <axis xyz="0 1 0"/>
+    <axis xyz="0 0 -1"/>
   </joint>
   <gazebo reference="right_wheel">

Commit message: Imu sesor dded to gazebo

File: description/robot_core.xacro (robot description, xacro)
@@ -245,3 +245,74 @@
     <mu2>0.01</mu2>
   </gazebo>
+  <!-- Define the IMU Link -->
+  <link name="imu_link">
+    <visual>
+      <geometry>
+        <box size="0.05 0.05 0.02"/>
+      </geometry>
+    </visual>
+    <inertial>
+      <mass value="0.01"/>
+      <inertia ixx="0.0001" ixy="0" ixz="0" iyy="0.0001" iyz="0" izz="0.0001"/>
+    </inertial>
+  </link>
+  <!-- Fix IMU to the Base -->
+  <joint name="imu_joint" type="fixed">
+    <parent link="base_link"/>
+    <child link="imu_link"/>
+    <origin xyz="0 0 0.05" rpy="0 0 0"/>
+  </joint>
+  <!-- Gazebo Sensor Plugin for IMU -->
+  <gazebo reference="imu_link">
+    <sensor name="imu_sensor" type="imu">
+      <always_on>true</always_on>
+      <update_rate>100</update_rate>
+      <topic>imu</topic>
+      <imu>
+        <angular_velocity>
+          <x>
+            <noise type="gaussian">
+              <mean>0</mean>
+              <stddev>0.009</stddev>
+            </noise>
+          </x>
+          <y>
+            <noise type="gaussian">
+              <mean>0</mean>
+              <stddev>0.009</stddev>
+            </noise>
+          </y>
+          <z>
+            <noise type="gaussian">
+              <mean>0</mean>
+              <stddev>0.009</stddev>
+            </noise>
+          </z>
+        </angular_velocity>
+        <linear_acceleration>
+          <x>
+            <noise type="gaussian">
+              <mean>0</mean>
+              <stddev>0.021</stddev>
+            </noise>
+          </x>
+          <y>
+            <noise type="gaussian">
+              <mean>0</mean>
+              <stddev>0.021</stddev>
+            </noise>
+          </y>
+          <z>
+            <noise type="gaussian">
+              <mean>0</mean>
+              <stddev>0.021</stddev>
+            </noise>
+          </z>
+        </linear_acceleration>
+      </imu>
+      <plugin filename="gz-sim-imu-system" name="gz::sim::systems::Imu">
+        <frame_id>imu_link</frame_id>
+      </plugin>
+    </sensor>
+  </gazebo>
 </robot>
